File: Kicad/Keeb_small_symetrical_hotswap_left/Keeb.kicad_sch (KiCad schematic)
At the start: 32 parts, among them J1 TYPE-C-31-M-12, J2 B2B-XH-A_LF__SN_, SW1 CherryMX, SW10 CherryMX, SW11 CherryMX, SW13 CherryMX, SW14 CherryMX, SW15 CherryMX, SW16 CherryMX, SW17 CherryMX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

Commit message: Switched footprint to copper plater one to give an opiton of soldering switches directly
Parts:
- SW1, SW10, SW11, SW13, SW14, SW15, SW16, SW17, SW18, SW19, SW2, SW20, SW3, SW4, SW5, SW6, SW7, SW8, SW9: footprint ScottoKeebs_Hotswap:Hotswap_MX_1.00u -> ScottoKeebs_Hotswap:Hotswap_MX_Plated_1.00u_Smaller_hole
Changed lines of the file:
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@@
       (effects (font (size 1.27 1.27)))
     )
-    (property "Footprint" "ScottoKeebs_Hotswap:Hotswap_MX_1.00u" (at 113.03 61.595 0)
+    (property "Footprint" "ScottoKeebs_Hotswap:Hotswap_MX_Plated_1.00u_Smaller_hole" (at 113.03 61.595 0)
       (effects (font (size 1.27 1.27)) hide)
     )
@@
       (effects (font (size 1.27 1.27)))
     )
-    (property "Footprint" "ScottoKeebs_Hotswap:Hotswap_MX_1.00u" (at 125.73 61.595 0)
+    (property "Footprint" "ScottoKeebs_Hotswap:Hotswap_MX_Plated_1.00u_Smaller_hole" (at 125.73 61.595 0)
       (effects (font (size 1.27 1.27)) hide)
     )
@@
       (effects (font (size 1.27 1.27)))
     )
-    (property "Footprint" "ScottoKeebs_Hotswap:Hotswap_MX_1.00u" (at 138.43 61.595 0)
+    (property "Footprint" "ScottoKeebs_Hotswap:Hotswap_MX_Plated_1.00u_Smaller_hole" (at 138.43 61.595 0)
       (effects (font (size 1.27 1.27)) hide)
     )
@@
       (effects (font (size 1.27 1.27)))
     )
-    (property "Footprint" "ScottoKeebs_Hotswap:Hotswap_MX_1.00u" (at 151.13 61.595 0)
+    (property "Footprint" "ScottoKeebs_Hotswap:Hotswap_MX_Plated_1.00u_Smaller_hole" (at 151.13 61.595 0)
       (effects (font (size 1.27 1.27)) hide)
     )
@@
       (effects (font (size 1.27 1.27)))
     )
-    (property "Footprint" "ScottoKeebs_Hotswap:Hotswap_MX_1.00u" (at 163.83 61.595 0)
+    (property "Footprint" "ScottoKeebs_Hotswap:Hotswap_MX_Plated_1.00u_Smaller_hole" (at 163.83 61.595 0)
       (effects (font (size 1.27 1.27)) hide)
     )
@@
       (effects (font (size 1.27 1.27)))
     )
-    (property "Footprint" "ScottoKeebs_Hotswap:Hotswap_MX_1.00u" (at 113.03 71.755 0)
+    (property "Footprint" "ScottoKeebs_Hotswap:Hotswap_MX_Plated_1.00u_Smaller_hole" (at 113.03 71.755 0)
       (effects (font (size 1.27 1.27)) hide)
     )
@@
       (effects (font (size 1.27 1.27)))
     )
-    (property "Footprint" "ScottoKeebs_Hotswap:Hotswap_MX_1.00u" (at 125.73 71.755 0)
+    (property "Footprint" "ScottoKeebs_Hotswap:Hotswap_MX_Plated_1.00u_Smaller_hole" (at 125.73 71.755 0)
       (effects (font (size 1.27 1.27)) hide)
     )
@@
       (effects (font (size 1.27 1.27)))
     )
-    (property "Footprint" "ScottoKeebs_Hotswap:Hotswap_MX_1.00u" (at 138.43 71.755 0)
+    (property "Footprint" "ScottoKeebs_Hotswap:Hotswap_MX_Plated_1.00u_Smaller_hole" (at 138.43 71.755 0)
       (effects (font (size 1.27 1.27)) hide)
     )
@@
       (effects (font (size 1.27 1.27)))
     )
-    (property "Footprint" "ScottoKeebs_Hotswap:Hotswap_MX_1.00u" (at 151.13 71.755 0)
+    (property "Footprint" "ScottoKeebs_Hotswap:Hotswap_MX_Plated_1.00u_Smaller_hole" (at 151.13 71.755 0)
       (effects (font (size 1.27 1.27)) hide)
     )
@@
       (effects (font (size 1.27 1.27)))
     )
-    (property "Footprint" "ScottoKeebs_Hotswap:Hotswap_MX_1.00u" (at 163.83 71.755 0)
+    (property "Footprint" "ScottoKeebs_Hotswap:Hotswap_MX_Plated_1.00u_Smaller_hole" (at 163.83 71.755 0)
       (effects (font (size 1.27 1.27)) hide)
     )
@@
       (effects (font (size 1.27 1.27)))
     )
-    (property "Footprint" "ScottoKeebs_Hotswap:Hotswap_MX_1.00u" (at 113.03 84.455 0)
+    (property "Footprint" "ScottoKeebs_Hotswap:Hotswap_MX_Plated_1.00u_Smaller_hole" (at 113.03 84.455 0)
       (effects (font (size 1.27 1.27)) hide)
     )
@@
       (effects (font (size 1.27 1.27)))
     )
-    (property "Footprint" "ScottoKeebs_Hotswap:Hotswap_MX_1.00u" (at 125.73 84.455 0)
+    (property "Footprint" "ScottoKeebs_Hotswap:Hotswap_MX_Plated_1.00u_Smaller_hole" (at 125.73 84.455 0)
       (effects (font (size 1.27 1.27)) hide)
     )
@@
       (effects (font (size 1.27 1.27)))
     )
-    (property "Footprint" "ScottoKeebs_Hotswap:Hotswap_MX_1.00u" (at 138.43 84.455 0)
+    (property "Footprint" "ScottoKeebs_Hotswap:Hotswap_MX_Plated_1.00u_Smaller_hole" (at 138.43 84.455 0)
       (effects (font (size 1.27 1.27)) hide)
     )
@@
       (effects (font (size 1.27 1.27)))
     )
-    (property "Footprint" "ScottoKeebs_Hotswap:Hotswap_MX_1.00u" (at 151.13 84.455 0)
+    (property "Footprint" "ScottoKeebs_Hotswap:Hotswap_MX_Plated_1.00u_Smaller_hole" (at 151.13 84.455 0)
       (effects (font (size 1.27 1.27)) hide)
     )
@@
       (effects (font (size 1.27 1.27)))
     )
-    (property "Footprint" "ScottoKeebs_Hotswap:Hotswap_MX_1.00u" (at 163.83 84.455 0)
+    (property "Footprint" "ScottoKeebs_Hotswap:Hotswap_MX_Plated_1.00u_Smaller_hole" (at 163.83 84.455 0)
       (effects (font (size 1.27 1.27)) hide)
     )
@@
       (effects (font (size 1.27 1.27)))
     )
-    (property "Footprint" "ScottoKeebs_Hotswap:Hotswap_MX_1.00u" (at 151.13 97.155 0)
+    (property "Footprint" "ScottoKeebs_Hotswap:Hotswap_MX_Plated_1.00u_Smaller_hole" (at 151.13 97.155 0)
       (effects (font (size 1.27 1.27)) hide)
     )
@@
       (effects (font (size 1.27 1.27)))
     )
-    (property "Footprint" "ScottoKeebs_Hotswap:Hotswap_MX_1.00u" (at 163.83 97.155 0)
+    (property "Footprint" "ScottoKeebs_Hotswap:Hotswap_MX_Plated_1.00u_Smaller_hole" (at 163.83 97.155 0)
       (effects (font (size 1.27 1.27)) hide)
     )
@@
       (effects (font (size 1.27 1.27)))
     )
-    (property "Footprint" "ScottoKeebs_Hotswap:Hotswap_MX_1.00u" (at 137.16 97.155 0)
+    (property "Footprint" "ScottoKeebs_Hotswap:Hotswap_MX_Plated_1.00u_Smaller_hole" (at 137.16 97.155 0)
       (effects (font (size 1.27 1.27)) hide)
     )
@@
       (effects (font (size 1.27 1.27)))
     )
-    (property "Footprint" "ScottoKeebs_Hotswap:Hotswap_MX_1.00u" (at 123.19 97.155 0)
-      (effects (font (size 1.27 1.27)) hide)
-    )
+    (property "Footprint" "ScottoKeebs_Hotswap:Hotswap_MX_Plated_1.00u_Smaller_hole" (at 123.19 97.155 0)
+      (effects (font (size 1.27 1.27)) hide)
+    )
