File: Kicad/Keeb_small_symetrical_hotswap_left/Keeb.kicad_pcb (KiCad board)
At the start: 2 copper layers, 96.2 x 98.1 mm, 32 parts, among them J1 TYPE-C-31-M-12, J2 B2B-XH-A_LF__SN_, SW1 CherryMX, SW10 CherryMX, SW11 CherryMX, SW13 CherryMX, SW14 CherryMX, SW15 CherryMX, SW16 CherryMX, SW17 CherryMX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

Commit message: Almost dome with right half
Parts:
- moved H9 27.6 mm to (167.8, 127.5)
Routing:
- net GND: track 606.6 -> 605.9 mm
