File: Kicad/Keeb_small_symetrical_hotswap_right/Keeb.kicad_sch (KiCad schematic)
At the start: 28 parts, among them J1 TYPE-C-31-M-12, SW1 CherryMX, SW10 CherryMX, SW11 CherryMX, SW13 CherryMX, SW14 CherryMX, SW15 CherryMX, SW16 CherryMX, SW17 CherryMX, SW18 CherryMX, SW19 CherryMX, SW20 CherryMX, SW3 CherryMX, SW4 CherryMX, SW5 CherryMX, SW6 CherryMX, SW7 CherryMX, SW8 CherryMX, SW9 CherryMX, U1 Pico

Commit message: Almost dome with right half
Parts:
- removed H6: MountingHole, MountingHole:MountingHole_3.2mm_M3, symbol Mechanical:MountingHole
- added H9: MountingHole, MountingHole:MountingHole_3.2mm_M3, symbol Mechanical:MountingHole
- added J2: B2B-XH-A_LF__SN_, Connectors_user:JST_B2B-XH-A_LF__SN_, symbol B2B-XH-A_LF__SN_:B2B-XH-A_LF__SN_
- added S1: DS01-254-L-01BE, DIP:SW_DS01-254-L-01BE, symbol DS01-254-L-01BE:DS01-254-L-01BE
- added SW2: CherryMX, ScottoKeebs_Hotswap:Hotswap_MX_Plated_1.00u_Smaller_hole, symbol Keeb-rescue:CherryMX-CherryMX
- added U2: KY-040, KY-040:KY-040-PORT, symbol KY-040:KY-040
- SW1, SW10, SW11, SW13, SW14, SW15, SW16, SW17, SW18, SW19, SW20, SW3, SW4, SW5, SW6, SW7, SW8, SW9: footprint ScottoKeebs_Hotswap:Hotswap_MX_1.00u -> ScottoKeebs_Hotswap:Hotswap_MX_Plated_1.00u_Smaller_hole
- U1: footprint MCU_RaspberryPi_and_Boards:RPi_Pico_SMD_TH_NO_HOLES -> MCU_RaspberryPi_and_Boards:RPi_Pico_SMD_TH_NO_BACK_HOLES
Connections:
- net 0: now also SW20.2; no longer J1.A5 (CC1), J1.A8 (SBU1)
- net 1: now also SW1.1; no longer J1.A6 (DP1), J1.A7 (DN1)
- net 10: now also SW14.2
- net 12: now also SW17.2; no longer SW14.2
- net 14: now also J1.B6 (DP2), J1.B7 (DN2)
- net 15: now also J1.A6 (DP1), J1.A7 (DN1)
- net 19: now also SW6.1; no longer SW8.2
- net 2: now also J1.A5 (CC1), J1.A8 (SBU1); no longer J1.B6 (DP2), J1.B7 (DN2)
- net 20: now also SW7.1; no longer SW7.2
- net 21: now also SW8.1; no longer SW6.2
- net 22: now also SW2.1
- net 28: now also SW5.1; no longer SW5.2
- net 3: now also SW19.2
- net 3v3: now also J1.A4_B9 (VBUS), J1.B4_A9 (VBUS), U2.VCC; no longer J1.B5 (CC2), J1.B8 (SBU2)
- net 4: now also SW16.1; no longer SW1.1
- net 5: now also SW18.2; no longer SW16.1
- net 6: no longer SW20.1
- net 7: now also U2.CLK; no longer SW19.1
- net 8: now also U2.DT; no longer SW18.1
- net 9: now also U2.SW; no longer SW17.1
- net GND: now also SW17.1, SW18.1, SW19.1, SW20.1, SW5.2, SW6.2, SW7.2, SW8.2, U1.33 (AGND), U1.8 (GND), S1.1A, SW2.2, U2.GND; no longer SW17.2, SW18.2, SW19.2, SW20.2, SW5.1, SW6.1, SW7.1, SW8.1
- net VSYS: now also J1.B5 (CC2), J1.B8 (SBU2), J2.1; no longer J1.A4_B9 (VBUS), J1.B4_A9 (VBUS)
- new net: J2.2, S1.1B
